File: homeCenter.sch (KiCad schematic (older format))
At the start: 44 parts, among them U1 CH340K

Commit message: update
Parts:
- added C?: 4.7u, symbol Device:C
- added J?: Conn_01x01_Female, symbol Connector:Conn_01x01_Female
- added U4: FengNiaoR3, kay:FengNiaoR3, symbol kay:FengNiaoR3
- IRM1: renamed from IRM?; symbol kay:IRM-H638T_TR2(DX) -> homeCenter-rescue:IRM-H638T_TR2(DX)-kay
- gave numbers to parts that had none: 42
Connections:
- net labels added: 433M_DAT
- wire segments 109 -> 120
Other:
- note added: "Power"
- moved on the sheet: C8, Q2, Q3, R14, R15, R16, U1

Commit message: update
Parts:
- removed C8: 1u, symbol Device:C
- removed D10, D8: ESD9B5.0ST5G, Diode_SMD:D_SOD-923, symbol Diode:ESD9B5.0ST5G
- removed J?: Conn_01x01_Female, symbol Connector:Conn_01x01_Female
- removed Q2, Q3: S8050, Package_TO_SOT_THT:TO-92_Inline, symbol Transistor_BJT:S8050
- removed R14, R15, R16: 10K, symbol Device:R
- removed U1: CH340K, kay:ESSOP-10, symbol kay:CH340K
- added D2, D3: LED, LED_SMD:LED_0603_1608Metric_Castellated, symbol Device:LED
- added J1, J2: sensor, Connector_PinHeader_2.54mm:PinHeader_1x02_P2.54mm_Vertical, symbol Connector:Conn_01x02_Male
- added J3: mcu_en, Capacitor_SMD:C_0504_1310Metric_Pad0.83x1.28mm_HandSolder, symbol Connector:Conn_01x02_Male
- added J4: Conn_01x01_Male, Connector_PinHeader_2.54mm:PinHeader_1x01_P2.54mm_Vertical, symbol Connector:Conn_01x01_Male
- added R3, R4: 47K, Resistor_SMD:R_0603_1608Metric, symbol Device:R
- C1: renamed from C2; footprint (none) -> Capacitor_SMD:C_0603_1608Metric
- C2: renamed from C3; footprint (none) -> Capacitor_SMD:C_0603_1608Metric
- C3: renamed from C4; footprint (none) -> Capacitor_SMD:C_0603_1608Metric
- C4: renamed from C5; footprint (none) -> Capacitor_SMD:C_0603_1608Metric
- C5: renamed from C6; footprint (none) -> Capacitor_SMD:C_0603_1608Metric
- C6: renamed from C7; footprint (none) -> Capacitor_SMD:C_0603_1608Metric
- C7: renamed from C?; footprint (none) -> Capacitor_SMD:C_0603_1608Metric
- C8: renamed from C1; footprint (none) -> Capacitor_SMD:C_0603_1608Metric
- D1: footprint Diode_SMD:D_SMB -> Diode_SMD:D_SOD-523
- D10: renamed from D9; footprint LED_SMD:LED_1206_3216Metric -> kay:LED-SMD_L3.0-W2.7-RD
- D11: footprint LED_SMD:LED_1206_3216Metric -> kay:LED-SMD_L3.0-W2.7-RD
- D4: renamed from D2; footprint LED_SMD:LED_1206_3216Metric -> kay:LED-SMD_L3.0-W2.7-RD
- D5: renamed from D3; footprint LED_SMD:LED_1206_3216Metric -> kay:LED-SMD_L3.0-W2.7-RD
- D6: renamed from D4; footprint LED_SMD:LED_1206_3216Metric -> kay:LED-SMD_L3.0-W2.7-RD
- D7: renamed from D5; footprint LED_SMD:LED_1206_3216Metric -> kay:LED-SMD_L3.0-W2.7-RD
- D8: renamed from D6; footprint LED_SMD:LED_1206_3216Metric -> kay:LED-SMD_L3.0-W2.7-RD
- D9: renamed from D7; footprint LED_SMD:LED_1206_3216Metric -> kay:LED-SMD_L3.0-W2.7-RD
- F1: footprint (none) -> Fuse:Fuse_1206_3216Metric_Castellated
- P1: footprint (none) -> Connector_USB:USB_C_Receptacle_HRO_TYPE-C-31-M-12
- Q1: footprint Package_TO_SOT_THT:TO-92_Inline -> Package_TO_SOT_SMD:SOT-23
- R1: renamed from R10; footprint (none) -> Resistor_SMD:R_0603_1608Metric
- R10: renamed from R6; footprint (none) -> Resistor_SMD:R_0603_1608Metric
- R11: renamed from R7; footprint (none) -> Resistor_SMD:R_0603_1608Metric
- R12: renamed from R8; footprint (none) -> Resistor_SMD:R_0603_1608Metric
- R13: renamed from R9; footprint (none) -> Resistor_SMD:R_0603_1608Metric
- R14: renamed from R12; footprint (none) -> Resistor_SMD:R_0603_1608Metric
- R15: renamed from R13; footprint (none) -> Resistor_SMD:R_0603_1608Metric
- R2: renamed from R11; footprint (none) -> Resistor_SMD:R_0603_1608Metric
- R5: renamed from R2; footprint (none) -> Resistor_SMD:R_0603_1608Metric
- R6: renamed from R1; footprint (none) -> Resistor_SMD:R_0603_1608Metric
- R7: renamed from R3; footprint (none) -> Resistor_SMD:R_0603_1608Metric
- R8: renamed from R4; footprint (none) -> Resistor_SMD:R_0603_1608Metric
- R9: renamed from R5; footprint (none) -> Resistor_SMD:R_0603_1608Metric
- renumbered U2 to U1, U3 to U2, U4 to U3
Connections:
- net labels added: SENSOR0, SENSOR1, TEST_LED0
- net labels removed: USB_N, USB_P
- wire segments 120 -> 102
- no-connect marks 1 -> 10
Other:
- note added: "433M"
- note added: "ESP32"
- note added: "IR\n"
- note added: "OTHERS\n"
- note added: "SENSOR"
- moved on the sheet: C1, C2, C3, C4, C5, C6, C7, C8, D1, D10, D11, D4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
