File: homeCenter.kicad_sch (KiCad schematic)
At the start: 39 parts, among them J1 sensor, J2 sensor, J3 M_SERIAL, J4 mcu_en, J5 Conn_01x01_Male, P1 USB_C_Plug_USB2.0, Q1 S8050, U1 AMS1117-3.3, U2 ESP32-WROOM-32, U3 FengNiaoR3

Commit message: pcb
Parts:
- removed Q1: S8050, Package_TO_SOT_SMD:SOT-23, symbol Transistor_BJT:S8050
- added Q1: Q_NPN_BEC, Package_TO_SOT_SMD:SOT-23, symbol Device:Q_NPN_BEC
- renumbered TP2 to 3V1, TP1 to 5V1
Connections:
- net 433M_DAT: now also U2.36 (IO22); no longer U2.14 (IO12)
- net GND: now also Q1.2 (E)
- net IR_RX0: now also U2.27 (IO16); no longer U2.16 (IO13)
- net SENSOR1: now also J1.2 (Pin_2), U2.26 (IO4); no longer J2.2 (Pin_2), U2.27 (IO16)
- net SENSOR2: now reaches U2.37 (IO23)
- net SENSOR2: now also J2.2 (Pin_2)
- net at D4.1 (K), D5.1 (K), D6.1 (K)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: now also Q1.3 (C)
- net at R6.2, R8.2: now also Q1.1 (B)
- net SENSOR0: no longer names the net of U2.23 (IO15)
- net SENSOR0: no longer J1.2 (Pin_2)
- no-connect marks 12 -> 14
Changed lines of the file:
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@@
   (no_connect (at 146.05 76.2))
   (no_connect (at 146.05 78.74))
+  (no_connect (at 176.53 40.64))
+  (no_connect (at 176.53 58.42))
   (wire (pts (xy 25.4 76.2) (xy 33.02 76.2))
     (stroke (width 0) (type solid) (color 0 0 0 0))
@@
     (stroke (width 0) (type solid) (color 0 0 0 0))
   )
-  (wire (pts (xy 176.53 50.8) (xy 186.69 50.8))
-    (stroke (width 0) (type solid) (color 0 0 0 0))
-  )
-  (wire (pts (xy 176.53 53.34) (xy 186.69 53.34))
+  (wire (pts (xy 176.53 45.72) (xy 186.69 45.72))
     (stroke (width 0) (type solid) (color 0 0 0 0))
   )
@@
     (stroke (width 0) (type solid) (color 0 0 0 0))
   )
-  (wire (pts (xy 176.53 58.42) (xy 186.69 58.42))
-    (stroke (width 0) (type solid) (color 0 0 0 0))
-  )
   (wire (pts (xy 176.53 60.96) (xy 186.69 60.96))
+    (stroke (width 0) (type solid) (color 0 0 0 0))
+  )
+  (wire (pts (xy 176.53 73.66) (xy 186.69 73.66))
+    (stroke (width 0) (type solid) (color 0 0 0 0))
+  )
+  (wire (pts (xy 176.53 76.2) (xy 186.69 76.2))
     (stroke (width 0) (type solid) (color 0 0 0 0))
   )
@@
     (effects (font (size 2.54 2.54)) (justify left bottom))
   )
-  (label "SENSOR0" (at 27.94 149.86 0)
-    (effects (font (size 1.27 1.27)) (justify left bottom))
-  )
-  (label "SENSOR1" (at 27.94 162.56 0)
+  (label "SENSOR1" (at 27.94 149.86 0)
+    (effects (font (size 1.27 1.27)) (justify left bottom))
+  )
+  (label "SENSOR2" (at 27.94 162.56 0)
     (effects (font (size 1.27 1.27)) (justify left bottom))
   )
@@
     (effects (font (size 1.27 1.27)) (justify left bottom))
   )
-  (label "433M_DAT" (at 177.8 50.8 0)
-    (effects (font (size 1.27 1.27)) (justify left bottom))
-  )
-  (label "IR_RX0" (at 177.8 53.34 0)
+  (label "SENSOR1" (at 177.8 45.72 0)
     (effects (font (size 1.27 1.27)) (justify left bottom))
   )
@@
     (effects (font (size 1.27 1.27)) (justify left bottom))
   )
-  (label "SENSOR0" (at 177.8 58.42 0)
-    (effects (font (size 1.27 1.27)) (justify left bottom))
-  )
-  (label "SENSOR1" (at 177.8 60.96 0)
+  (label "IR_RX0" (at 177.8 60.96 0)
+    (effects (font (size 1.27 1.27)) (justify left bottom))
+  )
+  (label "433M_DAT" (at 177.8 73.66 0)
+    (effects (font (size 1.27 1.27)) (justify left bottom))
+  )
+  (label "SENSOR2" (at 177.8 76.2 0)
     (effects (font (size 1.27 1.27)) (justify left bottom))
   )
@@
   (symbol (lib_id "Connector:TestPoint") (at 40.64 95.25 0) (unit 1)
     (in_bom yes) (on_board yes) (fields_autoplaced)
-    (property "Reference" "TP1" (id 0) (at 42.0371 92.5 0)
+    (property "Reference" "5V1" (id 0) (at 42.0371 92.5 0)
       (effects (font (size 1.27 1.27)) (justify left))
     )
@@
   (symbol (lib_id "Connector:TestPoint") (at 74.93 95.25 0) (unit 1)
     (in_bom yes) (on_board yes) (fields_autoplaced)
-    (property "Reference" "TP2" (id 0) (at 76.3271 92.5 0)
+    (property "Reference" "3V1" (id 0) (at 76.3271 92.5 0)
       (effects (font (size 1.27 1.27)) (justify left))
     )
@@
     (pin "2")
   )
-  (symbol (lib_id "Transistor_BJT:S8050") (at 243.84 88.9 0) (mirror x) (unit 1)
-    (in_bom yes) (on_board yes)
-    (property "Reference" "Q1" (id 0) (at 248.666 87.7316 0)
-      (effects (font (size 1.27 1.27)) (justify left))
-    )
-    (property "Value" "S8050" (id 1) (at 248.666 90.043 0)
-      (effects (font (size 1.27 1.27)) (justify left))
-    )
-    (property "Footprint" "Package_TO_SOT_SMD:SOT-23" (id 2) (at 248.92 86.995 0)
-      (effects (font (size 1.27 1.27) italic) (justify left) hide)
-    )
-    (property "Datasheet" "http://www.unisonic.com.tw/datasheet/S8050.pdf" (id 3) (at 243.84 88.9 0)
-      (effects (font (size 1.27 1.27)) (justify left) hide)
+  (symbol (lib_id "Device:Q_NPN_BEC") (at 243.84 88.9 0) (unit 1)
+    (in_bom yes) (on_board yes) (fields_autoplaced)
+    (property "Reference" "Q1" (id 0) (at 248.6915 87.9915 0)
+      (effects (font (size 1.27 1.27)) (justify left))
+    )
+    (property "Value" "Q_NPN_BEC" (id 1) (at 248.6915 90.7666 0)
+      (effects (font (size 1.27 1.27)) (justify left))
+    )
+    (property "Footprint" "Package_TO_SOT_SMD:SOT-23" (id 2) (at 248.92 86.36 0)
+      (effects (font (size 1.27 1.27)) hide)
+    )
+    (property "Datasheet" "~" (id 3) (at 243.84 88.9 0)
+      (effects (font (size 1.27 1.27)) hide)
     )
     (pin "1")
@@
       (reference "#PWR014") (unit 1) (value "GND") (footprint "")
     )
+    (path "/1f5ce82f-3fd7-4053-8adb-fc8fc66958ed"
+      (reference "3V1") (unit 1) (value "3V3") (footprint "TestPoint:TestPoint_Pad_D1.0mm")
+    )
+    (path "/8a3b2b4e-5877-4d53-a830-bd90843f7e33"
+      (reference "5V1") (unit 1) (value "5V") (footprint "TestPoint:TestPoint_Pad_D1.0mm")
+    )
     (path "/c6f7fa14-603b-491d-a9ce-a267cd658b5c"
       (reference "C1") (unit 1) (value "22u") (footprint "kay:CAP-SMD_L3.2-W1.6-RD")
@@
       (reference "P1") (unit 1) (value "USB_C_Plug_USB2.0") (footprint "Connector_USB:USB_C_Receptacle_HRO_TYPE-C-31-M-12")
     )
-    (path "/00000000-0000-0000-0000-000060de168d"
-      (reference "Q1") (unit 1) (value "S8050") (footprint "Package_TO_SOT_SMD:SOT-23")
+    (path "/ba3691a0-2b65-4679-8115-9b711ba2c902"
+      (reference "Q1") (unit 1) (value "Q_NPN_BEC") (footprint "Package_TO_SOT_SMD:SOT-23")
     )
     (path "/00000000-0000-0000-0000-000060d16fe7"
@@
       (reference "R10") (unit 1) (value "47") (footprint "Resistor_SMD:R_0603_1608Metric")
     )
-    (path "/8a3b2b4e-5877-4d53-a830-bd90843f7e33"
-      (reference "TP1") (unit 1) (value "5V") (footprint "TestPoint:TestPoint_Pad_D1.0mm")
-    )
-    (path "/1f5ce82f-3fd7-4053-8adb-fc8fc66958ed"
-      (reference "TP2") (unit 1) (value "3V3") (footprint "TestPoint:TestPoint_Pad_D1.0mm")
-    )
     (path "/00000000-0000-0000-0000-000060d0ce50"

Commit message: v0.2
Parts:
- renumbered 5V1 to TP1, 3V1 to TP2
Changed lines of the file:
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@@
   (symbol (lib_id "Connector:TestPoint") (at 40.64 95.25 0) (unit 1)
     (in_bom yes) (on_board yes) (fields_autoplaced)
-    (property "Reference" "5V1" (id 0) (at 42.0371 92.5 0)
+    (property "Reference" "TP1" (id 0) (at 42.0371 92.5 0)
       (effects (font (size 1.27 1.27)) (justify left))
     )
@@
   (symbol (lib_id "Connector:TestPoint") (at 74.93 95.25 0) (unit 1)
     (in_bom yes) (on_board yes) (fields_autoplaced)
-    (property "Reference" "3V1" (id 0) (at 76.3271 92.5 0)
+    (property "Reference" "TP2" (id 0) (at 76.3271 92.5 0)
       (effects (font (size 1.27 1.27)) (justify left))
     )
@@
       (reference "#PWR014") (unit 1) (value "GND") (footprint "")
     )
-    (path "/1f5ce82f-3fd7-4053-8adb-fc8fc66958ed"
-      (reference "3V1") (unit 1) (value "3V3") (footprint "TestPoint:TestPoint_Pad_D1.0mm")
-    )
-    (path "/8a3b2b4e-5877-4d53-a830-bd90843f7e33"
-      (reference "5V1") (unit 1) (value "5V") (footprint "TestPoint:TestPoint_Pad_D1.0mm")
-    )
     (path "/c6f7fa14-603b-491d-a9ce-a267cd658b5c"
       (reference "C1") (unit 1) (value "22u") (footprint "kay:CAP-SMD_L3.2-W1.6-RD")
@@
       (reference "R10") (unit 1) (value "47") (footprint "Resistor_SMD:R_0603_1608Metric")
     )
+    (path "/8a3b2b4e-5877-4d53-a830-bd90843f7e33"
+      (reference "TP1") (unit 1) (value "5V") (footprint "TestPoint:TestPoint_Pad_D1.0mm")
+    )
+    (path "/1f5ce82f-3fd7-4053-8adb-fc8fc66958ed"
+      (reference "TP2") (unit 1) (value "3V3") (footprint "TestPoint:TestPoint_Pad_D1.0mm")
+    )
     (path "/00000000-0000-0000-0000-000060d0ce50"
